File: Power.kicad_sch (KiCad schematic)
At the start: 43 parts, among them J10 Conn_01x02_Socket, J22 Conn_01x02_Socket, J23 Conn_01x02_Socket, J24 Conn_01x02_Socket, Q1 NMOS, U10 INA219AxD, U11 TLV62569ADRL, U15 TPS60400DBV, U9 INA219AxD

Commit message: didnt save?
Parts:
- removed C20: 4u7, Capacitor_SMD:C_0603_1608Metric, symbol Device:C
- removed C21: 22u, Capacitor_SMD:C_0603_1608Metric, symbol Device:C
- removed C51, C54, C55: DNP, Capacitor_SMD:C_0603_1608Metric, symbol Device:C
- removed D10: D, Diode_SMD:D_1206_3216Metric, symbol Device:D
- removed D5: LED, LED_SMD:LED_0603_1608Metric, symbol Device:LED
- removed J10: Conn_01x02_Socket, Connector_Phoenix_SPT:PhoenixContact_SPT_2.5_2-H-5.0_1x02_P5.0mm_Horizontal, symbol Connector:Conn_01x02_Socket
- removed L1: 1u, Inductor_SMD:L_Bourns-SRN8040_8x8.15mm, symbol Device:L
- removed Q1: NMOS, Package_TO_SOT_SMD:TO-252-3_TabPin2, symbol Simulation_SPICE:NMOS
- removed R31: 10R, Resistor_SMD:R_0603_1608Metric, symbol Device:R
- removed R32: 10k, Resistor_SMD:R_0603_1608Metric, symbol Device:R
- removed R40: 453k, Resistor_SMD:R_0603_1608Metric, symbol Device:R
- removed R41: 100k, Resistor_SMD:R_0603_1608Metric, symbol Device:R
- removed R42: 2m, Resistor_SMD:R_0603_1608Metric, symbol Device:R
- removed R43: 330, Resistor_SMD:R_0603_1608Metric, symbol Device:R
- removed U11: TLV62569ADRL, Package_TO_SOT_SMD:SOT-563, symbol Regulator_Switching:TLV62569ADRL
Other:
- note removed: "BUCK CONVERTER 5V-3.3V"
- note removed: "LED MATRIX PWR CTRL"
- note removed: "https://webench.ti.com/power-designer/switching-regulator/export/12?noparams=0"
