File: Wireless.kicad_sch (KiCad schematic)
At the start: 37 parts, among them J11 Conn_01x02_Pin, J16 Conn_01x04_Pin, J17 Conn_01x04_Pin, SW6 SW_Push, SW7 SW_Push, U14 ESP32-C3FH4, Y2 40MHz

Commit message: gettind rid of esp32
Parts:
- removed AE1: Antenna_Shield, RF_Antenna:Texas_SWRA117D_2.4GHz_Left, symbol Device:Antenna_Shield
- removed C26, C27: 22p, Capacitor_SMD:C_0603_1608Metric, symbol Device:C
- removed C28, C29, C30, C31: DNP, Capacitor_SMD:C_0402_1005Metric, symbol Device:C
- removed C32, C34, C35, C36, C37, C45: 100n, Capacitor_SMD:C_0603_1608Metric, symbol Device:C
- removed C33, C39: 1u, Capacitor_SMD:C_0603_1608Metric, symbol Device:C
- removed C38: 10u, Capacitor_SMD:C_0603_1608Metric, symbol Device:C
- removed D9: LED, LED_SMD:LED_0603_1608Metric, symbol Device:LED
- removed J11: Conn_01x02_Pin, Connector_PinHeader_2.54mm:PinHeader_1x02_P2.54mm_Vertical, symbol Connector:Conn_01x02_Pin
- removed J16, J17: Conn_01x04_Pin, Connector_PinHeader_2.54mm:PinHeader_1x04_P2.54mm_Vertical, symbol Connector:Conn_01x04_Pin
- removed L2, L3: DNP, Inductor_SMD:L_0402_1005Metric, symbol Device:L
- removed L4: 2n, Inductor_SMD:L_0603_1608Metric_Pad1.05x0.95mm_HandSolder, symbol Device:L
- removed R54: 330, Resistor_SMD:R_0603_1608Metric, symbol Device:R
- removed R55, R56, R57, R58: 0R, Resistor_SMD:R_0603_1608Metric, symbol Device:R
- removed R59, R60, R78, R79: 10k, Resistor_SMD:R_0603_1608Metric, symbol Device:R
- removed R76: 1k, Resistor_SMD:R_0603_1608Metric, symbol Device:R
- removed SW6, SW7: SW_Push, Button_Switch_THT:SW_PUSH_6mm, symbol Switch:SW_Push
- removed U14: ESP32-C3FH4, Package_DFN_QFN:QFN-32-1EP_5x5mm_P0.5mm_EP3.45x3.45mm, symbol PCM_Espressif:ESP32-C3
- removed Y2: 40MHz, Crystal:Crystal_SMD_ECS_CSM3X-2Pin_7.6x4.1mm, symbol Device:Crystal
Connections:
- no-connect marks 11 -> 0
Other:
- note removed: "ANTENNA"
- note removed: "BOOT BUTTON"
- note removed: "BREAKOUTS"
- note removed: "CRYSTAL OSC"
- note removed: "ESP32"
- note removed: "PWR CAPS"
- note removed: "RESET BUTTON"
- note removed: "TEST LED"
